File: schematics/FootSensor/FootSensorV1.brd (EAGLE design)
At the start: 30.5 x 12.7 mm, 22 parts, among them IC1 MCP6V261, P1 PAD_THROUGH1, P2 PAD_THROUGH1, P3 PAD_THROUGH1, P4 PAD_THROUGH1, P5 PAD_THROUGH1, P6 PAD_THROUGH1, P7 PAD_THROUGH1, P8 PAD_THROUGH1, P9 PAD_THROUGH1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

Commit message: no message
Parts:
- moved LED3 22.9 mm to (-5.12, 0.70)
- moved R8 22.9 mm to (-2.90, 1.81)
- moved IC1 22.9 mm to (-5.28, -1.52)
- moved P5 22.9 mm to (-7.98, 4.03)
- moved P6 22.9 mm to (-6.23, 4.83)
- moved P7 22.9 mm to (-4.33, 4.83)
- moved P8 22.9 mm to (-2.58, 4.03)
- moved P9 22.9 mm to (-1.31, 2.60)
- moved Q1 22.9 mm to (-5.32, 0.70)
- moved R3 22.9 mm to (-8.61, 1.47)
- moved R4 22.9 mm to (-5.28, 1.97)
- moved R5 22.9 mm to (-7.50, 1.49)
- moved R6 22.9 mm to (-7.18, 0.70)
- moved R7 22.9 mm to (-3.06, 0.70)
- moved P1 17.2 mm to (-21.0, 2.41)
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Routing:
- net GND: track 10.5 -> 9.26 mm
- removed copper zone on layer 1, net GND
- removed copper zone on layer 16, net GND
Other:
- board size 30.5 x 12.7 mm -> 22.1 x 10.1 mm
