File: schematics/FootSensor/FootSensor.sch (EAGLE design)
At the start: 22 parts, among them IC1 MCP6V261, P1 PAD_THROUGH1, P2 PAD_THROUGH1, P3 PAD_THROUGH1, P4 PAD_THROUGH1, P5 PAD_THROUGH1, P6 PAD_THROUGH1, P7 PAD_THROUGH1, P8 PAD_THROUGH1, P9 PAD_THROUGH1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

Commit message: Corrected silkscreen on Footsensor
Other:
- note added: "Opamp PCB"
- note removed: "Komparator PCB"
- moved on the sheet: Q1
Changed lines of the file:
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@@
 <?xml version="1.0" encoding="utf-8"?>
 <!DOCTYPE eagle SYSTEM "eagle.dtd">
-<eagle version="6.5.0">
+<eagle version="9.6.2">
 <drawing>
 <settings>
 <setting alwaysvectorfont="no"/>
+<setting keepoldvectorfont="yes"/>
 <setting verticaltext="up"/>
 </settings>
@@
 <text x="-22.86" y="187.96" size="1.778" layer="94">Aperture</text>
 <text x="-71.12" y="132.08" size="1.778" layer="94">LED PCB</text>
-<text x="87.63" y="177.8" size="1.778" layer="94">Komparator PCB</text>
+<text x="87.63" y="177.8" size="1.778" layer="94">Opamp PCB</text>
 <circle x="-92.71" y="157.48" radius="59.5141" width="0.1524" layer="94"/>
 <circle x="55.88" y="157.48" radius="59.5141" width="0.1524" layer="94"/>
@@
 <text x="-105.41" y="134.62" size="1.016" layer="94">display LED</text>
 <text x="-59.69" y="146.05" size="1.016" layer="94">Light barrier LED</text>
-<wire x1="-76.2" y1="173.99" x2="-39.37" y2="173.99" width="0.1524" layer="94" style="shortdash"/>
+<wire x1="-77.47" y1="173.99" x2="-39.37" y2="173.99" width="0.1524" layer="94" style="shortdash"/>
 <wire x1="-39.37" y1="173.99" x2="-38.1" y2="172.72" width="0.1524" layer="94" style="shortdash"/>
 <wire x1="-38.1" y1="172.72" x2="-38.1" y2="146.05" width="0.1524" layer="94" style="shortdash"/>
@@
 <wire x1="-78.74" y1="146.05" x2="-78.74" y2="172.72" width="0.1524" layer="94" style="shortdash"/>
 <wire x1="-78.74" y1="172.72" x2="-77.47" y2="173.99" width="0.1524" layer="94" style="shortdash"/>
-<wire x1="-77.47" y1="173.99" x2="-76.2" y2="173.99" width="0.1524" layer="94" style="shortdash"/>
 <wire x1="-128.27" y1="172.72" x2="-127" y2="173.99" width="0.1524" layer="94" style="shortdash"/>
 <wire x1="-127" y1="173.99" x2="-93.98" y2="173.99" width="0.1524" layer="94" style="shortdash"/>
@@
 <wire x1="-93.98" y1="124.46" x2="-127" y2="124.46" width="0.1524" layer="94" style="shortdash"/>
 <wire x1="-127" y1="124.46" x2="-128.27" y2="125.73" width="0.1524" layer="94" style="shortdash"/>
-<wire x1="-128.27" y1="125.73" x2="-128.27" y2="170.18" width="0.1524" layer="94" style="shortdash"/>
-<wire x1="-128.27" y1="170.18" x2="-128.27" y2="171.45" width="0.1524" layer="94" style="shortdash"/>
-<wire x1="-128.27" y1="171.45" x2="-128.27" y2="172.72" width="0.1524" layer="94" style="shortdash"/>
+<wire x1="-128.27" y1="125.73" x2="-128.27" y2="172.72" width="0.1524" layer="94" style="shortdash"/>
 </plain>
 <instances>
@@
 <attribute name="VALUE" x="33.02" y="106.68" size="0.8128" layer="96" font="vector" ratio="12"/>
 </instance>
-<instance part="Q1" gate="G$1" x="5.08" y="162.56" smashed="yes">
-<attribute name="NAME" x="2.286" y="168.148" size="0.8128" layer="95" font="vector" ratio="12"/>
-<attribute name="VALUE" x="2.286" y="155.194" size="0.8128" layer="95" font="vector" ratio="12"/>
+<instance part="Q1" gate="G$1" x="10.16" y="162.56" smashed="yes">
+<attribute name="NAME" x="7.366" y="168.148" size="0.8128" layer="95" font="vector" ratio="12"/>
+<attribute name="VALUE" x="7.366" y="155.194" size="0.8128" layer="95" font="vector" ratio="12"/>
 </instance>
 <instance part="P+3" gate="G$1" x="27.94" y="172.72" smashed="yes">
@@
 <instance part="PORT19" gate="G$1" x="-59.69" y="156.21" smashed="yes" rot="R180"/>
 <instance part="PORT19" gate="G$2" x="-69.85" y="156.21" smashed="yes" rot="R180"/>
-<instance part="Y1" gate="G$1" x="-165.1" y="55.88"/>
+<instance part="Y1" gate="G$1" x="-165.1" y="55.88" smashed="yes">
+<attribute name="LAST_DATE_TIME" x="153.43" y="65.88" size="1.27" layer="100"/>
+<attribute name="DRAWING_NAME" x="103.9" y="60.88" size="1.27" layer="100"/>
+<attribute name="SHEET" x="212.43" y="65.88" size="1.27" layer="100"/>
+</instance>
 </instances>
 <busses>
@@
 <pinref part="P+3" gate="G$1" pin="+3,3V"/>
 <wire x1="27.94" y1="172.72" x2="27.94" y2="167.64" width="0.1524" layer="91"/>
-<wire x1="30.48" y1="167.64" x2="43.18" y2="167.64" width="0.1524" layer="91"/>
-<wire x1="30.48" y1="167.64" x2="27.94" y2="167.64" width="0.1524" layer="91"/>
+<wire x1="27.94" y1="167.64" x2="43.18" y2="167.64" width="0.1524" layer="91"/>
 <junction x="27.94" y="167.64"/>
-<wire x1="27.94" y1="167.64" x2="12.7" y2="167.64" width="0.1524" layer="91"/>
+<wire x1="27.94" y1="167.64" x2="17.78" y2="167.64" width="0.1524" layer="91"/>
 <label x="49.022" y="167.64" size="0.8128" layer="95"/>
 </segment>
@@
 </segment>
 <segment>
+<wire x1="-119.38" y1="190.5" x2="-109.22" y2="190.5" width="0.1524" layer="91"/>
+<label x="-128.524" y="190.754" size="0.8128" layer="95"/>
 <pinref part="P1" gate="G$1" pin="1"/>
-<wire x1="-109.22" y1="195.58" x2="-109.22" y2="198.12" width="0.1524" layer="91"/>
-<wire x1="-109.22" y1="198.12" x2="-109.22" y2="193.04" width="0.1524" layer="91"/>
-<wire x1="-119.38" y1="190.5" x2="-109.22" y2="190.5" width="0.1524" layer="91"/>
-<wire x1="-109.22" y1="190.5" x2="-109.22" y2="193.04" width="0.1524" layer="91"/>
-<label x="-128.524" y="190.754" size="0.8128" layer="95"/>
+<wire x1="-109.22" y1="195.58" x2="-109.22" y2="190.5" width="0.1524" layer="91"/>
 </segment>
 </net>
@@
 <pinref part="Q1" gate="G$1" pin="E"/>
 <pinref part="R3" gate="G$1" pin="2"/>
-<wire x1="12.7" y1="157.48" x2="27.94" y2="157.48" width="0.1524" layer="91"/>
+<wire x1="17.78" y1="157.48" x2="27.94" y2="157.48" width="0.1524" layer="91"/>
 <wire x1="27.94" y1="157.48" x2="27.94" y2="147.32" width="0.1524" layer="91"/>
 <pinref part="IC1" gate="A" pin="2"/>

Commit message: Printed Toe, Foot & Thigh
Parts:
- R4: value S10K_0603 -> S51K_0603; device joshi:S10K_0603 -> joshi:S51K_0603
- R5: value S20K_0603 -> S5.1K_0603; device joshi:S20K_0603 -> joshi:S5.1K_0603
Changed lines of the file:
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@@
 <part name="R6" library="joshi" deviceset="S51R_0603" device=""/>
 <part name="R7" library="joshi" deviceset="S51R_0603" device=""/>
-<part name="R4" library="joshi" deviceset="S10K_0603" device=""/>
-<part name="R5" library="joshi" deviceset="S20K_0603" device=""/>
+<part name="R4" library="joshi" deviceset="S51K_0603" device=""/>
+<part name="R5" library="joshi" deviceset="S5.1K_0603" device=""/>
 <part name="P7" library="Connectors" deviceset="PAD_THROUGH" device="1"/>
 <part name="P5" library="Connectors" deviceset="PAD_THROUGH" device="1"/>
