Commit message: cleanup description

File: description/solo12.urdf (robot description, URDF)
Before this commit: robot solo, 17 links, 16 joints
Links:
- link FL_FOOT: geometry collision mesh filename=../../../description/meshes/stl/foot.stl; visual mesh filename=../../../description/meshes/stl/foot.stl
- link FL_LOWER_LEG: geometry collision mesh filename=../../../description/meshes/stl/lower_leg_left_side.stl; visual mesh filename=../../../description/meshes/stl/lower_leg_left_side.stl
- link FL_SHOULDER: geometry collision mesh filename=../../../description/meshes/stl/hip_fe_fl.stl; visual mesh filename=../../../description/meshes/stl/hip_fe_fl.stl
- link FL_UPPER_LEG: geometry collision mesh filename=../../../description/meshes/stl/upper_leg_left_side.stl; visual mesh filename=../../../description/meshes/stl/upper_leg_left_side.stl
- link FR_FOOT: geometry collision mesh filename=../../../description/meshes/stl/foot.stl; visual mesh filename=../../../description/meshes/stl/foot.stl
- link FR_LOWER_LEG: geometry collision mesh filename=../../../description/meshes/stl/lower_leg_right_side.stl; visual mesh filename=../../../description/meshes/stl/lower_leg_right_side.stl
- link FR_SHOULDER: geometry collision mesh filename=../../../description/meshes/stl/hip_fe_fr.stl; visual mesh filename=../../../description/meshes/stl/hip_fe_fr.stl
- link FR_UPPER_LEG: geometry collision mesh filename=../../../description/meshes/stl/upper_leg_right_side.stl; visual mesh filename=../../../description/meshes/stl/upper_leg_right_side.stl
- link HL_FOOT: geometry collision mesh filename=../../../description/meshes/stl/foot.stl; visual mesh filename=../../../description/meshes/stl/foot.stl
- link HL_LOWER_LEG: geometry collision mesh filename=../../../description/meshes/stl/lower_leg_left_side.stl; visual mesh filename=../../../description/meshes/stl/lower_leg_left_side.stl
- link HL_SHOULDER: geometry collision mesh filename=../../../description/meshes/stl/hip_fe_hl.stl; visual mesh filename=../../../description/meshes/stl/hip_fe_hl.stl
- link HL_UPPER_LEG: geometry collision mesh filename=../../../description/meshes/stl/upper_leg_left_side.stl; visual mesh filename=../../../description/meshes/stl/upper_leg_left_side.stl
- link HR_FOOT: geometry collision mesh filename=../../../description/meshes/stl/foot.stl; visual mesh filename=../../../description/meshes/stl/foot.stl
- link HR_LOWER_LEG: geometry collision mesh filename=../../../description/meshes/stl/lower_leg_right_side.stl; visual mesh filename=../../../description/meshes/stl/lower_leg_right_side.stl
- link HR_SHOULDER: geometry collision mesh filename=../../../description/meshes/stl/hip_fe_hr.stl; visual mesh filename=../../../description/meshes/stl/hip_fe_hr.stl
- link HR_UPPER_LEG: geometry collision mesh filename=../../../description/meshes/stl/upper_leg_right_side.stl; visual mesh filename=../../../description/meshes/stl/upper_leg_right_side.stl
- link base_link: geometry collision mesh filename=../../../description/meshes/stl/base.stl; visual mesh filename=../../../description/meshes/stl/base.stl

File: description/solo12.urdf.xacro (robot description, xacro)
@@ -25,5 +25,5 @@
         <origin xyz="0 0 0" rpy="0 0 0" />
         <geometry>
-          <mesh filename="package://robot_properties_solo/resources/meshes/${mesh_ext}/solo12/solo_12_base.${mesh_ext}"/>
+          <mesh filename="package://robot_properties_solo/resources/meshes/${mesh_ext}/solo_12_base.${mesh_ext}"/>
         </geometry>
         <material name="${color_name}">
@@ -35,5 +35,5 @@
         <origin xyz="0 0 0" rpy="0 0 0" />
         <geometry>
-          <mesh filename="package://robot_properties_solo/resources/meshes/${mesh_ext}/solo12/solo_12_base.${mesh_ext}"/>
+          <mesh filename="package://robot_properties_solo/resources/meshes/${mesh_ext}/solo_12_base.${mesh_ext}"/>
         </geometry>
         <material name="${color_name}">
