File: schematics/vestibular/vestibular.brd (EAGLE design)
At the start: 43.2 x 23.8 mm, 15 parts, among them IC2 SN75C3232, P2 Cerebellum, P4 3DM-GX3-25

Commit message: no message
Parts:
- R11: value 22k -> 27k
Changed lines of the file:
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@@
 <attribute name="VALUE" x="-1.524" y="16.764" size="1.27" layer="27" ratio="10" rot="R180"/>
 </element>
-<element name="R11" library="rcl" library_urn="urn:adsk.eagle:library:334" package="0204/7" package3d_urn="urn:adsk.eagle:package:23498/2" value="22k" x="-10.795" y="12.7" smashed="yes" rot="R90">
+<element name="R11" library="rcl" library_urn="urn:adsk.eagle:library:334" package="0204/7" package3d_urn="urn:adsk.eagle:package:23498/2" value="27k" x="-10.795" y="12.7" smashed="yes" rot="R90">
 <attribute name="NAME" x="-10.1854" y="11.43" size="0.9906" layer="25" ratio="10" rot="R90"/>
 <attribute name="POPULARITY" value="79" x="-10.795" y="12.7" size="1.778" layer="27" rot="R90" display="off"/>
