File: schematics/cerebellar/cerebellar V1.0.brd (EAGLE design)
At the start: 98.4 x 91.1 mm, 68 parts, among them CON2 ODrive1, CON4 Odrive3, CON5 ODrive4, CON6 Odrive2, CON7 ODrive5, CON8 ODrive6, IC3 LTC7001, P1 Foot1, P10 SPI2, P11 Foot2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

Commit message: buffersize in UART7 for less checksum errors
Connections:
- removed net MAG_EN: U$1.9-OUT1C
Changed lines of the file:
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@@
 <via x="84.4296" y="18.3896" extent="1-16" drill="0.35"/>
-</signal>
-<signal name="MAG_EN">
-<contactref element="U$1" pad="9-OUT1C"/>
 </signal>
 <signal name="MAG_INT">
