File: schematics/cerebellar/cerebellar V1.1.sch (EAGLE design)
At the start: 68 parts, among them CON1 ODRV2, CON2 ODRV1, CON3 ODRV3, CON4 ODRV4, CON5 ODRV5, CON6 ODRV6, IC3 LTC7001, P1 Foot1, P10 SPI2, P11 Foot2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

Commit message: Schematics with power supply and INA works
Parts:
- added R6: 100k, rcl:R-EU_0204/7
- C1, C19, C2, C3: device rcl:C-EU025-025X050 -> rcl:C-EU050-024X044
- C4: device rcl:C-EU025-025X050 -> rcl:CPOL-EUE2-4
- P3: value SPI2 -> SPI1; device jst-ph:JST-PH5 -> jst-ph:JST-PH6
Connections:
- removed net N$9: U$1.6-OUT1D, U$8.SHDN
- new net SHDN: R6.1, U$1.6-OUT1D, U$8.SHDN
- net +3.3V: now also C4.+; no longer C4.1
- net GND: now also C4.-, R6.2, U$8.GND; no longer C4.2
- net N$7: now also P3.6
Other:
- moved on the sheet: C1, C2, C3

Commit message: MOSFET Driver tested
Parts:
- removed P10: SPI2, jst-ph:JST-PH5
- added P17: SPI2, jst-ph:JST-PH6
- U$2, U$3, U$5: value IRF2804 -> IRF2804-BACK; device IRF2804:IRF2804 -> IRF2804:IRF2804-BACK
Connections:
- net N$10 renamed INP
- net N$26 renamed TS
- net N$4 renamed TGUP
- removed net N$18: SJ5.1, U2.IN-
- removed net N$7: P3.6, U$1.3V3-3
- new net N$9: P17.6, P3.6, U$1.3V3-3
- new net PMS+: C25.+, C26.1, R20.1, SJ5.1, U$7.VS, U2.IN-
- net CS1: now also P17.4; no longer P10.4
- net GND: now also P17.1; no longer P10.1
- net MISO1: now also P17.2; no longer P10.2
- net MOSI1: now also P17.3; no longer P10.3
- net SCK1: now also P17.5; no longer P10.5
- net V+: no longer C25.+, C26.1, R20.1, U$7.VS

Commit message: buffersize in UART7 for less checksum errors
Connections:
- net N$9 renamed T3.3V
- removed net MAG_EN: U$1.9-OUT1C
Changed lines of the file:
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@@
 <segment>
 <pinref part="P14" gate="G$1" pin="2"/>
-<wire x1="248.92" y1="36.83" x2="242.57" y2="36.83" width="0.1524" layer="91"/>
+<wire x1="248.92" y1="36.83" x2="238.76" y2="36.83" width="0.1524" layer="91"/>
 <label x="242.57" y="36.83" size="1.778" layer="95"/>
 </segment>
 <segment>
-<wire x1="248.92" y1="12.7" x2="234.95" y2="12.7" width="0.1524" layer="91"/>
-<label x="234.95" y="12.7" size="1.778" layer="95"/>
 <pinref part="P16" gate="G$1" pin="3"/>
+<wire x1="248.92" y1="12.7" x2="237.49" y2="12.7" width="0.1524" layer="91"/>
+<label x="237.49" y="12.7" size="1.778" layer="95"/>
 </segment>
 </net>
@@
 <wire x1="163.83" y1="34.29" x2="163.83" y2="11.43" width="0.1524" layer="91"/>
 <wire x1="163.83" y1="11.43" x2="149.86" y2="11.43" width="0.1524" layer="91"/>
+<label x="149.86" y="11.43" size="1.778" layer="95"/>
+<wire x1="163.83" y1="34.29" x2="248.92" y2="34.29" width="0.1524" layer="91"/>
 <pinref part="P14" gate="G$1" pin="1"/>
-<wire x1="248.92" y1="34.29" x2="163.83" y2="34.29" width="0.1524" layer="91"/>
-<label x="149.86" y="11.43" size="1.778" layer="95"/>
+<label x="233.68" y="34.29" size="1.778" layer="95"/>
 </segment>
 </net>
@@
 </segment>
 <segment>
-<wire x1="248.92" y1="15.24" x2="234.95" y2="15.24" width="0.1524" layer="91"/>
-<label x="234.95" y="15.24" size="1.778" layer="95"/>
 <pinref part="P16" gate="G$1" pin="4"/>
+<wire x1="248.92" y1="15.24" x2="237.49" y2="15.24" width="0.1524" layer="91"/>
+<label x="237.49" y="15.24" size="1.778" layer="95"/>
 </segment>
 </net>
@@
 </segment>
 <segment>
-<wire x1="248.92" y1="17.78" x2="234.95" y2="17.78" width="0.1524" layer="91"/>
-<label x="234.95" y="17.78" size="1.778" layer="95"/>
 <pinref part="P16" gate="G$1" pin="5"/>
-</segment>
-</net>
-<net name="MAG_EN" class="0">
-<segment>
-<pinref part="U$1" gate="G$1" pin="9-OUT1C"/>
-<wire x1="149.86" y1="8.89" x2="163.83" y2="8.89" width="0.1524" layer="91"/>
-<label x="149.86" y="8.89" size="1.778" layer="95"/>
+<wire x1="248.92" y1="17.78" x2="236.22" y2="17.78" width="0.1524" layer="91"/>
+<label x="237.49" y="17.78" size="1.778" layer="95"/>
 </segment>
 </net>
@@
 </segment>
 <segment>
-<wire x1="248.92" y1="7.62" x2="229.87" y2="7.62" width="0.1524" layer="91"/>
-<label x="234.95" y="7.62" size="1.778" layer="95"/>
 <pinref part="P16" gate="G$1" pin="1"/>
+<wire x1="248.92" y1="7.62" x2="236.22" y2="7.62" width="0.1524" layer="91"/>
+<label x="236.22" y="7.62" size="1.778" layer="95"/>
 </segment>
 </net>
@@
 <junction x="52.07" y="177.8"/>
 <wire x1="52.07" y1="175.26" x2="52.07" y2="177.8" width="0.1524" layer="91"/>
+<pinref part="C3" gate="G$1" pin="1"/>
+<pinref part="C4" gate="G$1" pin="+"/>
+<pinref part="P16" gate="G$1" pin="2"/>
 <wire x1="248.92" y1="10.16" x2="232.41" y2="10.16" width="0.1524" layer="91"/>
 <junction x="232.41" y="10.16"/>
-<pinref part="P16" gate="G$1" pin="2"/>
-<pinref part="C3" gate="G$1" pin="1"/>
-<pinref part="C4" gate="G$1" pin="+"/>
 </segment>
 </net>
@@
 </segment>
 </net>
-<net name="N$9" class="0">
+<net name="T3.3V" class="0">
 <segment>
 <pinref part="P17" gate="A" pin="6"/>
@@
 <wire x1="184.15" y1="85.09" x2="134.62" y2="85.09" width="0.1524" layer="91"/>
 <junction x="184.15" y="12.7"/>
-</segment>
-</net>
+<label x="201.93" y="13.97" size="1.778" layer="95"/>
+</segment>
+</net>

Commit message: Added LED Power Manager
Parts:
- removed R8: 100, rcl:R-EU_0204/7
- R20: value 25k -> 100k
- U$4: value MAX769L -> MAX869L
Connections:
- net N$47 renamed SWTCH
- removed net N$3: P4.1, R8.2
- removed net N$6: R8.1, U$4.OUT
- new net LED+: P4.1, U$4.OUT
Changed lines of the file:
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@@
 <part name="L2" library="rcl" library_urn="urn:adsk.eagle:library:334" deviceset="L-EU" device="IRF-3" package3d_urn="urn:adsk.eagle:package:23536/1" value="10uH"/>
 <part name="U$7" library="TLF50211EL" deviceset="TLF50211EL" device=""/>
-<part name="R20" library="rcl" library_urn="urn:adsk.eagle:library:334" deviceset="R-EU_" device="0204/7" package3d_urn="urn:adsk.eagle:package:23498/2" value="25k"/>
+<part name="R20" library="rcl" library_urn="urn:adsk.eagle:library:334" deviceset="R-EU_" device="0204/7" package3d_urn="urn:adsk.eagle:package:23498/2" value="100k"/>
 <part name="R21" library="rcl" library_urn="urn:adsk.eagle:library:334" deviceset="R-EU_" device="0204/7" package3d_urn="urn:adsk.eagle:package:23498/2" value="100k"/>
 <part name="D3" library="diode" library_urn="urn:adsk.eagle:library:210" deviceset="ZENER-DIODE" device="DO41Z10" package3d_urn="urn:adsk.eagle:package:43341/1" value="Z 5.1V 1A"/>
@@
 <part name="SUPPLY5" library="supply2" library_urn="urn:adsk.eagle:library:372" deviceset="GND" device=""/>
 <part name="P14" library="jst-ph" deviceset="JST-PH5" device="" value="IMU"/>
-<part name="U$4" library="MAX869" deviceset="MAX769L" device=""/>
+<part name="U$4" library="MAX869" deviceset="MAX769L" device="" value="MAX869L"/>
 <part name="SUPPLY2" library="supply2" library_urn="urn:adsk.eagle:library:372" deviceset="GND" device=""/>
 <part name="R1" library="rcl" library_urn="urn:adsk.eagle:library:334" deviceset="R-EU_" device="0204/7" package3d_urn="urn:adsk.eagle:package:23498/2" value="6.8k"/>
 <part name="P4" library="jst-ph" deviceset="JST-PH2" device="" value="LED"/>
-<part name="R8" library="rcl" library_urn="urn:adsk.eagle:library:334" deviceset="R-EU_" device="0204/7" package3d_urn="urn:adsk.eagle:package:23498/2" value="100"/>
 <part name="U$8" library="LT1763" deviceset="LT1763" device=""/>
 <part name="P16" library="jst-ph" deviceset="JST-PH5" device="" value="MAG"/>
@@
 <attribute name="NAME" x="392.43" y="89.408" size="1.778" layer="95" rot="R180"/>
 <attribute name="VALUE" x="392.43" y="100.076" size="1.778" layer="96" rot="R180"/>
-</instance>
-<instance part="R8" gate="G$1" x="346.71" y="92.71" smashed="yes">
-<attribute name="NAME" x="342.9" y="94.2086" size="1.778" layer="95"/>
-<attribute name="VALUE" x="342.9" y="89.408" size="1.778" layer="96"/>
 </instance>
 <instance part="U$8" gate="G$1" x="39.37" y="170.18" smashed="yes"/>
@@
 </segment>
 </net>
-<net name="N$47" class="0">
+<net name="SWTCH" class="0">
 <segment>
 <pinref part="U$7" gate="G$1" pin="EN"/>
@@
 <wire x1="-102.87" y1="193.04" x2="-156.21" y2="193.04" width="0.1524" layer="91"/>
 <junction x="-156.21" y="193.04"/>
+<label x="-156.21" y="149.86" size="1.778" layer="95"/>
 </segment>
 </net>
@@
 </segment>
 </net>
-<net name="N$6" class="0">
+<net name="LED+" class="0">
 <segment>
 <pinref part="U$4" gate="G$1" pin="OUT"/>
 <wire x1="341.63" y1="92.71" x2="334.01" y2="92.71" width="0.1524" layer="91"/>
-<pinref part="R8" gate="G$1" pin="1"/>
-</segment>
-</net>
-<net name="N$3" class="0">
-<segment>
-<pinref part="R8" gate="G$1" pin="2"/>
 <pinref part="P4" gate="G$1" pin="1"/>
-<wire x1="351.79" y1="92.71" x2="382.27" y2="92.71" width="0.1524" layer="91"/>
-</segment>
-</net>
+<wire x1="341.63" y1="92.71" x2="382.27" y2="92.71" width="0.1524" layer="91"/>
+<label x="375.92" y="92.71" size="1.778" layer="95"/>
+</segment>
+</net>

Commit message: improved schmeatics
Other:
- note added: "PWM LED, 5V, 2A"
- note added: "Sockets Display"
- note added: "Sockets IMU & MAG"
- note removed: "PWM LED, 2A"
- moved on the sheet: C2, C25, C26, C3, C4, C6, D2, D3, L2, LED1, P1, P11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
